Commit message: update

File: src/rl_demo/models/cube.urdf (robot description, URDF)
Before this commit: robot simple_object, 1 links, 0 joints
Links:
- link my_object: mass 1.0 -> 0.001; geometry collision box size=0.05 0.05 0.05; visual box size=0.05 0.05 0.05

File: src/rl_gazebo/urdf/rlbot.urdf.xacro (robot description, xacro)
@@ -8,5 +8,5 @@
     <!-- camera settings -->
     <xacro:include filename="$(find rl_gazebo)/urdf/rlbot.gazebo.xacro" />
-    <!-- arm -->
+    <!-- Arm -->
     <xacro:ur5_robot prefix="" joint_limited="false" transmission_hw_interface="$(arg transmission_hw_interface)"/>
     <link name="world" />
@@ -16,4 +16,9 @@
         <origin xyz="0.0 0.0 0.0" rpy="0.0 0.0 0.0" />
     </joint>
+    <!-- Gripper -->
+    <xacro:include filename="$(find robotiq_85_description)/urdf/robotiq_85_gripper.urdf.xacro" />
+    <xacro:robotiq_85_gripper prefix="" parent="tool0" >
+        <origin xyz="0.0 0.0 0.0" rpy="0 ${-pi/2} 0"/>
+    </xacro:robotiq_85_gripper>
     <!-- Camera -->
     <xacro:property name="camera_link" value="0.02" /> <!-- Size of square 'camera' box -->
@@ -40,6 +45,6 @@
     <joint name="camera_joint" type="fixed">
         <axis xyz="0 1 0" />
-        <origin xyz="-0.02 0.045 0" rpy="0 0 0"/>
-        <parent link="ee_link"/>
+        <origin xyz="0.02 0 0.045" rpy="0 0 0"/>
+        <parent link="gripper_base_link"/>
         <child link="camera_link"/>
     </joint>
